File: 500W-Mono-ClassAB-Amplifier.kicad_sch (KiCad schematic)
At the start: 0 parts

Commit message: Update to well-formed KiCad v7 schematic, PCB and project files (500W)
Parts:
- added R1: 10k, Resistors_SMD:R_0805, symbol Device:R
Changed lines of the file:
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@@
-(kicad_sch (version 20211014) (generator kicad_sch)
+(kicad_sch (version 20211014) (generator KiCad)
   (paper "A4")
   (title "500W-Mono-ClassAB-Amplifier")
   (date "2026-09-06")
-  (comment "Minimal valid KiCad v7 schematic for CI: contains one resistor from the standard Device library.")
-  (components
-    (comp (ref R1) (value "10k") (footprint "Resistors_SMD:R_0805") (lib_id "Device:R")
-      (unit 1)
-      (symbol "R")
-      (at 50 50)
-    )
+  (kicad_version "7.0.10")
+  (symbol (lib_id "Device:R")
+    (at 50 50)
+    (unit 1)
+    (tstamp 0x5F3759E0)
+    (property "Reference" "R1")
+    (property "Value" "10k")
+    (property "Footprint" "Resistors_SMD:R_0805")
+    (pin "1" (type passive) (at 0 0))
+    (pin "2" (type passive) (at 100 0))
   )
-  (nets
-    (net (code 1) (name "NET1")
-      (node (ref R1) (pin 1) (x 50) (y 50))
-      (node (ref R1) (pin 2) (x 70) (y 50))
-    )
+  (net (code 1) (name "NET1")
+    (node (ref R1) (pin 1) (x 50) (y 50))
+    (node (ref R1) (pin 2) (x 150) (y 50))
   )
 )
